File: hw2/HW2CHONG.brd (EAGLE design)
At the start: 50 x 50 mm, 23 parts

Commit message: HW2
Parts:
- moved U$7 0.63 mm to (45.7, 5.71)
Routing:
- net +3V3: track 119.9 -> 122.7 mm
- net N$13: track 20.1 -> 19.4 mm
- net N$12: track 25.2 -> 24.5 mm
Changed lines of the file:
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@@
 </class>
 </classes>
-<designrules name="default">
+<designrules name="SeeedStudio_2layer_DRU_no_angle_20140221">
 <description language="de">&lt;b&gt;EAGLE Design Rules&lt;/b&gt;
 &lt;p&gt;
@@
 necessary adjustments and save your customized
 design rules under a new name.</description>
+<description language="zh">&lt;b&gt;Seeed Studio EAGLE Design Rules&lt;/b&gt;
+</description>
 <param name="layerSetup" value="(1*16)"/>
-<param name="mtCopper" value="0.035mm 0.035mm 0.035mm 0.035mm 0.035mm 0.035mm 0.035mm 0.035mm 0.035mm 0.035mm 0.035mm 0.035mm 0.035mm 0.035mm 0.035mm 0.035mm"/>
-<param name="mtIsolate" value="1.5mm 0.15mm 0.2mm 0.15mm 0.2mm 0.15mm 0.2mm 0.15mm 0.2mm 0.15mm 0.2mm 0.15mm 0.2mm 0.15mm 0.2mm"/>
-<param name="mdWireWire" value="8mil"/>
-<param name="mdWirePad" value="8mil"/>
-<param name="mdWireVia" value="8mil"/>
-<param name="mdPadPad" value="8mil"/>
-<param name="mdPadVia" value="8mil"/>
-<param name="mdViaVia" value="8mil"/>
-<param name="mdSmdPad" value="8mil"/>
-<param name="mdSmdVia" value="8mil"/>
-<param name="mdSmdSmd" value="8mil"/>
+<param name="mtCopper" value="0.035mm 0.0175mm 0.035mm 0.035mm 0.035mm 0.035mm 0.035mm 0.035mm 0.035mm 0.035mm 0.035mm 0.035mm 0.035mm 0.035mm 0.0175mm 0.035mm"/>
+<param name="mtIsolate" value="1.5mm 1.1mm 0.2mm 0.15mm 0.2mm 0.15mm 0.2mm 0.15mm 0.2mm 0.15mm 0.2mm 0.15mm 0.2mm 0.15mm 0.2mm"/>
+<param name="mdWireWire" value="6mil"/>
+<param name="mdWirePad" value="6mil"/>
+<param name="mdWireVia" value="6mil"/>
+<param name="mdPadPad" value="6mil"/>
+<param name="mdPadVia" value="6mil"/>
+<param name="mdViaVia" value="6mil"/>
+<param name="mdSmdPad" value="0mil"/>
+<param name="mdSmdVia" value="0mil"/>
+<param name="mdSmdSmd" value="0mil"/>
 <param name="mdViaViaSameLayer" value="8mil"/>
 <param name="mnLayersViaInSmd" value="2"/>
-<param name="mdCopperDimension" value="40mil"/>
-<param name="mdDrill" value="8mil"/>
+<param name="mdCopperDimension" value="10mil"/>
+<param name="mdDrill" value="10mil"/>
 <param name="mdSmdStop" value="0mil"/>
-<param name="msWidth" value="10mil"/>
-<param name="msDrill" value="24mil"/>
-<param name="msMicroVia" value="9.99mm"/>
+<param name="msWidth" value="6mil"/>
+<param name="msDrill" value="12mil"/>
+<param name="msMicroVia" value="12mil"/>
 <param name="msBlindViaRatio" value="0.5"/>
 <param name="rvPadTop" value="0.25"/>
@@
 <param name="rlMinPadBottom" value="10mil"/>
 <param name="rlMaxPadBottom" value="20mil"/>
-<param name="rlMinViaOuter" value="8mil"/>
+<param name="rlMinViaOuter" value="6mil"/>
 <param name="rlMaxViaOuter" value="20mil"/>
-<param name="rlMinViaInner" value="8mil"/>
+<param name="rlMinViaInner" value="6mil"/>
 <param name="rlMaxViaInner" value="20mil"/>
 <param name="rlMinMicroViaOuter" value="4mil"/>
@@
 <param name="psTop" value="-1"/>
 <param name="psBottom" value="-1"/>
-<param name="psFirst" value="-1"/>
+<param name="psFirst" value="0"/>
 <param name="psElongationLong" value="100"/>
 <param name="psElongationOffset" value="100"/>
 <param name="mvStopFrame" value="1"/>
 <param name="mvCreamFrame" value="0"/>
-<param name="mlMinStopFrame" value="4mil"/>
-<param name="mlMaxStopFrame" value="4mil"/>
+<param name="mlMinStopFrame" value="2mil"/>
+<param name="mlMaxStopFrame" value="2mil"/>
 <param name="mlMinCreamFrame" value="0mil"/>
 <param name="mlMaxCreamFrame" value="0mil"/>
-<param name="mlViaStopLimit" value="0mil"/>
+<param name="mlViaStopLimit" value="100mil"/>
 <param name="srRoundness" value="0"/>
 <param name="srMinRoundness" value="0mil"/>
@@
 <param name="checkAngle" value="0"/>
 <param name="checkFont" value="1"/>
-<param name="checkRestrict" value="1"/>
+<param name="checkRestrict" value="0"/>
 <param name="useDiameter" value="13"/>
 <param name="maxErrors" value="50"/>
@@
 <element name="U$5" library="HW2LIBRARY" package="TO92" value="MCP1702" x="8.255" y="25.4" rot="R90"/>
 <element name="U$6" library="HW2LIBRARY" package="1X06" value="PICKIT3" x="14.605" y="48.26" rot="R180"/>
-<element name="U$7" library="HW2LIBRARY" package="USB-MB-H" value="USBMINIBU" x="45.72" y="5.08" rot="R180"/>
+<element name="U$7" library="HW2LIBRARY" package="USB-MB-H" value="USBMINIBU" x="45.72" y="5.715" rot="R180"/>
 <element name="U$8" library="HW2LIBRARY" package="1X08" value="M08LEFT" x="1.27" y="34.29" rot="R270"/>
 <element name="U$9" library="HW2LIBRARY" package="1X08" value="M08RIGHT" x="48.895" y="34.29" rot="R270"/>
@@
 <wire x1="34.925" y1="26.67" x2="29.845" y2="21.59" width="0.4064" layer="16"/>
 <wire x1="29.845" y1="21.59" x2="27.94" y2="21.59" width="0.4064" layer="16"/>
-<wire x1="17.145" y1="39.37" x2="35.56" y2="39.37" width="0.4064" layer="16"/>
 <wire x1="35.56" y1="39.37" x2="36.195" y2="39.37" width="0.4064" layer="16"/>
 <wire x1="36.195" y1="39.37" x2="38.1" y2="37.465" width="0.4064" layer="16"/>
@@
 <wire x1="15.24" y1="7.62" x2="15.24" y2="12.7" width="0.4064" layer="16"/>
 <wire x1="15.24" y1="12.7" x2="10.16" y2="17.78" width="0.4064" layer="16"/>
+<wire x1="17.145" y1="39.37" x2="18.415" y2="39.37" width="0.4064" layer="16"/>
+<wire x1="18.415" y1="39.37" x2="20.955" y2="41.91" width="0.4064" layer="16"/>
+<wire x1="20.955" y1="41.91" x2="34.29" y2="41.91" width="0.4064" layer="16"/>
+<wire x1="34.29" y1="41.91" x2="35.56" y2="40.64" width="0.4064" layer="16"/>
+<wire x1="35.56" y1="40.64" x2="35.56" y2="39.37" width="0.4064" layer="16"/>
 </signal>
 <signal name="GND">
@@
 <contactref element="U$7" pad="D-"/>
 <contactref element="U$1" pad="22"/>
-<wire x1="41.82" y1="4.28" x2="42.38" y2="4.28" width="0.4064" layer="16"/>
-<wire x1="42.38" y1="4.28" x2="43.815" y2="5.715" width="0.4064" layer="16"/>
-<wire x1="43.815" y1="5.715" x2="43.815" y2="6.985" width="0.4064" layer="16"/>
+<wire x1="41.82" y1="4.915" x2="42.38" y2="4.915" width="0.4064" layer="16"/>
+<wire x1="42.38" y1="4.915" x2="43.815" y2="6.35" width="0.4064" layer="16"/>
+<wire x1="43.815" y1="6.35" x2="43.815" y2="6.985" width="0.4064" layer="16"/>
 <wire x1="43.815" y1="6.985" x2="41.91" y2="8.89" width="0.4064" layer="16"/>
 <wire x1="41.91" y1="8.89" x2="41.91" y2="19.05" width="0.4064" layer="16"/>
@@
 <wire x1="38.735" y1="18.415" x2="38.735" y2="15.875" width="0.4064" layer="1"/>
 <via x="38.735" y="15.875" extent="1-16" drill="0.6"/>
-<wire x1="38.735" y1="15.875" x2="38.735" y2="5.715" width="0.4064" layer="16"/>
-<wire x1="38.735" y1="5.715" x2="39.37" y2="5.08" width="0.4064" layer="16"/>
-<wire x1="39.37" y1="5.08" x2="40.62" y2="5.08" width="0.4064" layer="16"/>
+<wire x1="38.735" y1="15.875" x2="38.735" y2="6.35" width="0.4064" layer="16"/>
+<wire x1="38.735" y1="6.35" x2="39.37" y2="5.715" width="0.4064" layer="16"/>
+<wire x1="39.37" y1="5.715" x2="40.62" y2="5.715" width="0.4064" layer="16"/>
 </signal>
 <signal name="N$14">
 <contactref element="U$7" pad="ID"/>
 <contactref element="U$1" pad="14"/>
-<wire x1="41.82" y1="5.88" x2="42.38" y2="5.88" width="0.4064" layer="1"/>
+<wire x1="41.82" y1="6.515" x2="42.38" y2="5.88" width="0.4064" layer="1"/>
 <wire x1="42.38" y1="5.88" x2="43.815" y2="4.445" width="0.4064" layer="1"/>
 <wire x1="43.815" y1="4.445" x2="43.815" y2="3.175" width="0.4064" layer="1"/>
@@
 <wire x1="7.62" y1="5.715" x2="6.35" y2="4.445" width="0.4064" layer="1"/>
 <wire x1="6.35" y1="4.445" x2="6.35" y2="2.54" width="0.4064" layer="1"/>
-<wire x1="40.62" y1="3.48" x2="38.43" y2="3.48" width="0.4064" layer="1"/>
-<wire x1="38.43" y1="3.48" x2="35.56" y2="6.35" width="0.4064" layer="1"/>
+<wire x1="40.62" y1="4.115" x2="38.43" y2="4.115" width="0.4064" layer="1"/>
+<wire x1="38.43" y1="4.115" x2="35.56" y2="6.35" width="0.4064" layer="1"/>
 <wire x1="48.895" y1="19.05" x2="48.26" y2="19.05" width="0.4064" layer="1"/>
 <wire x1="48.26" y1="19.05" x2="35.56" y2="6.35" width="0.4064" layer="1"/>
